Commit message: ver_0719_修改部分xacro

File: src/robo/urdf/car.xacro (robot description, xacro)
@@ -1,4 +1,6 @@
 <?xml version="1.0"?>
-<robot name="balancing_robot" xmlns:xacro="http://ros.org/wiki/xacro">
+<robot name="balancing_robot"
+    xmlns:xacro="http://ros.org/wiki/xacro">
+    <xacro:property name="pi" value="3.1415926"/>
     <xacro:property name="base_link_length" value="0.4"/>
     <xacro:property name="base_link_radius" value="0.01"/>
@@ -11,25 +13,54 @@
     <xacro:property name="UAV_y" value="0.4"/>
     <xacro:property name="UAV_z" value="0.05"/>
-    <material name="gray">
-        <color rgba="0.5 0.5 0.5 1.0"/>
+    <material name="red">
+        <color rgba="1.0 0.0 0.0 1.0"/>
+    </material>
+    <material name="green">
+        <color rgba="0.0 1.0 0.0 1.0"/>
     </material>
     <material name="blue">
-        <color rgba="0.0 0.0 0.8 1.0"/>
+        <color rgba="0.0 0.0 1.0 1.0"/>
+    </material>
+    <material name="yellow">
+        <color rgba="1.0 1.0 0.0 1.0"/>
+    </material>
+    <material name="cyan">
+        <color rgba="0.0 1.0 1.0 1.0"/>
+    </material>
+    <material name="orange">
+        <color rgba="1.0 0.5 0.0 1.0"/>
+    </material>
+    <material name="purple">
+        <color rgba="0.5 0.0 0.5 1.0"/>
     </material>
     <!-- Virtual linkage, as specifying inertia on the base_link is not supported -->
-    <link name="dummy_link"/>
+    <link name="dummy_link">
+        <visual>
+            <geometry>
+                <sphere radius="0.05"/>
+            </geometry>
+            <!-- <material name="dummy_link_color">
+                <color rgba="0.5 0.2 0.5 1" />
+            </material> -->
+            <!-- 这里是rviz显示的颜色 -->
+            <material name="red"/>
+        </visual>
+    </link>
+    <gazebo reference="dummy_link">
+        <material>Gazebo/Red</material>
+    </gazebo>
     <link name="base_link">
         <visual>
-            <origin rpy="1.5707 0 0"/>
             <geometry>
                 <cylinder radius="${base_link_radius}" length="${base_link_length}"/>
             </geometry>
-            <material name="gray"/>
+            <origin xyz="0 0 0" rpy="${pi/2} 0 0"/>
+            <material name="yellow"/>
         </visual>
         <collision>
-            <origin rpy="1.5707 0 0"/>
             <geometry>
                 <cylinder radius="${base_link_radius}" length="${base_link_length}"/>
             </geometry>
+            <origin xyz="0 0 0" rpy="${pi/2} 0 0"/>
         </collision>
         <inertial>
@@ -38,22 +69,26 @@
         </inertial>
     </link>
+    <gazebo reference="base_link">
+        <material>Gazebo/Yellow</material>
+    </gazebo>
     <joint name="dummy_to_base" type="fixed">
         <parent link="dummy_link"/>
         <child link="base_link"/>
+        <origin xyz="0 0 0" rpy="0 0 0" />
     </joint>
-    <xacro:macro name="wheel" params="param pos">
+    <xacro:macro name="wheel_func" params="direc pos">
         <link name="${pos}_wheel">
             <visual>
-                <origin xyz="0 0 0" rpy="1.5707 0 0"/>
                 <geometry>
                     <cylinder radius="${wheel_radius}" length="${wheel_width}"/>
                 </geometry>
-                <material name="blue"/>
+                <origin xyz="0 0 0" rpy="${pi/2} 0 0"/>
+                <material name="green"/>
             </visual>
             <collision>
-                <origin xyz="0 0 0" rpy="1.5707 0 0"/>
                 <geometry>
                     <cylinder radius="${wheel_radius}" length="${wheel_width}"/>
                 </geometry>
+                <origin xyz="0 0 0" rpy="${pi/2} 0 0"/>
             </collision>
             <inertial>
@@ -65,5 +100,5 @@
             <parent link="base_link"/>
             <child link="${pos}_wheel"/>
-            <origin xyz="0 ${param * base_link_length/2} 0"/>
+            <origin xyz="0 ${direc * base_link_length/2} 0" rpy="0 0 0"/>
             <axis xyz="0 1 0"/>
         </joint>
@@ -71,5 +106,5 @@
             <mu1 value="200"/>
             <mu2 value="100"/>
-            <material>Gazebo/Grey</material>
+            <material>Gazebo/Green</material>
         </gazebo>
         <transmission name="${pos}_wheel_trans">
@@ -83,19 +118,19 @@
         </transmission>
     </xacro:macro>
-    <xacro:wheel param="1" pos="left"/>
-    <xacro:wheel param="-1" pos="right"/>
+    <xacro:wheel_func direc="1" pos="left"/>
+    <xacro:wheel_func direc="-1" pos="right"/>
     <link name="support">
         <visual>
-            <origin xyz="0.0 0.0 0"/>
             <geometry>
                 <box size="${support_x} ${support_y} ${support_z}"/>
             </geometry>
-            <material name="gray"/>
+            <origin xyz="0 0 0"/>
+            <material name="blue"/>
         </visual>
         <collision>
-            <origin xyz="0.0 0.0 ${support_z/2}"/>
             <geometry>
                 <box size="${support_x} ${support_y} ${support_z}"/>
             </geometry>
+            <origin xyz="0 0 0"/>
         </collision>
         <inertial>
@@ -104,9 +139,13 @@
         </inertial>
     </link>
+    <gazebo reference="support">
+        <material>Gazebo/Blue</material>
+    </gazebo>
     <joint name="base_to_support" type="fixed">
         <parent link="base_link"/>
         <child link="support"/>
-        <origin xyz="0.0 0.0 ${support_z/2}"/>
+        <origin xyz="0 0 ${support_z/2}" rpy="${pi/2} 0 0"/>
     </joint>
+    <!--
     <link name="UAV">
         <visual name="">
@@ -156,4 +195,4 @@
             <pose>0 0 0 0 0 0</pose>
         </sensor>
-    </gazebo>
+    </gazebo> -->
 </robot>

Commit message: ver_0720_xacro理解完毕

File: src/robo/urdf/car.xacro (robot description, xacro)
@@ -34,9 +34,12 @@
         <color rgba="0.5 0.0 0.5 1.0"/>
     </material>
+    <material name="white">
+        <color rgba="1 1 1 1.0"/>
+    </material>
     <!-- Virtual linkage, as specifying inertia on the base_link is not supported -->
     <link name="dummy_link">
         <visual>
             <geometry>
-                <sphere radius="0.05"/>
+                <sphere radius="0.01"/>
             </geometry>
             <!-- <material name="dummy_link_color">
@@ -104,6 +107,6 @@
         </joint>
         <gazebo reference="${pos}_wheel">
-            <mu1 value="200"/>
-            <mu2 value="100"/>
+            <mu1 value="2"/>
+            <mu2 value="1"/>
             <material>Gazebo/Green</material>
         </gazebo>
@@ -145,20 +148,19 @@
         <parent link="base_link"/>
         <child link="support"/>
-        <origin xyz="0 0 ${support_z/2}" rpy="${pi/2} 0 0"/>
+        <origin xyz="0 0 ${support_z/2}" rpy="0 0 0"/>
     </joint>
-    <!--
     <link name="UAV">
         <visual name="">
-            <origin xyz="0.0 0.0 0"/>
             <geometry>
                 <box size="${UAV_x} ${UAV_y} ${UAV_z}"/>
             </geometry>
-            <material name="gray"/>
+            <origin xyz="0 0 0" rpy="0 0 0"/>
+            <material name="white"/>
         </visual>
         <collision>
-            <origin xyz="0.0 0.0 ${support_z}"/>
             <geometry>
                 <box size="${UAV_x} ${UAV_y} ${UAV_z}"/>
             </geometry>
+            <origin xyz="0 0 0" rpy="0 0 0"/>
         </collision>
         <inertial>
@@ -167,8 +169,11 @@
         </inertial>
     </link>
+    <gazebo reference="UAV">
+        <material>Gazebo/White</material>
+    </gazebo>
     <joint name="UAV_to_support" type="fixed">
         <parent link="support"/>
         <child link="UAV"/>
-        <origin xyz="0.0 0.0 ${support_z/2}"/>
+        <origin xyz="0 0 ${support_z/2}" rpy="0 0 0"/>
     </joint>
     <gazebo>
@@ -188,11 +193,11 @@
                 <bodyName>body_link</bodyName>
                 <updateRateHZ>50.0</updateRateHZ>
-                <gaussianNoise>0.0</gaussianNoise>
+                <gaussianNoise>0</gaussianNoise>
                 <xyzOffset>0 0 0</xyzOffset>
                 <rpyOffset>0 0 0</rpyOffset>
                 <frameName>imu_link</frameName>
             </plugin>
-            <pose>0 0 0 0 0 0</pose>
+            <pose>1 0 0 0 0 0</pose>
         </sensor>
-    </gazebo> -->
+    </gazebo>
 </robot>

Commit message: ver_0721_基本看完代码

File: src/robo/urdf/car.xacro (robot description, xacro)
@@ -78,5 +78,5 @@
         <parent link="dummy_link"/>
         <child link="base_link"/>
-        <origin xyz="0 0 0" rpy="0 0 0" />
+        <origin xyz="0 0 ${wheel_radius}" rpy="0 0 0" />
     </joint>
     <xacro:macro name="wheel_func" params="direc pos">
@@ -190,6 +190,5 @@
             <topic>__default_topic__</topic>
             <plugin filename="libgazebo_ros_imu_sensor.so" name="imu_plugin">
-                <topicName>imu/data</topicName>
-                <bodyName>body_link</bodyName>
+                <topicName>/imu/data</topicName>
                 <updateRateHZ>50.0</updateRateHZ>
                 <gaussianNoise>0</gaussianNoise>
